File: MCU.kicad_sch (KiCad schematic)
At the start: 6 parts, among them U1 STM32F446RETx

Commit message: added SWD connector
Parts:
- added J1: Conn_01x02_Pin, symbol Connector:Conn_01x02_Pin
- added J2, J4: Conn_01x06_Pin, symbol Connector:Conn_01x06_Pin
- added JP2: SolderJumper_2_Bridged, symbol Jumper:SolderJumper_2_Bridged
Connections:
- net GND: now also J1.2 (Pin_2), J2.3 (Pin_3)
- net VDD: now also JP1.1 (A)
- net VDD_STM: now also JP1.2 (B), J2.1 (Pin_1), JP2.2 (B)
- net NRST: now reaches U1.7 (NRST)
- net NRST: now also J2.5 (Pin_5)
- new net SWCLK: J2.2 (Pin_2)
- new net SWDIO: J2.4 (Pin_4)
- new net SWO: J2.6 (Pin_6)
- new net VDD_STM_EXT: J1.1 (Pin_1), JP2.1 (A)
Other:
- moved on the sheet: C1, C2, C3, JP1, R1
